File: extension_circuit_board/extension_circuit_board.kicad_pcb (KiCad board)
At the start: 2 copper layers, 95 x 72 mm, 6 parts, among them J1 AE_MRUSB_DIP, J2 Jetson_Nano_GPIO, J3 PiOLED 2x3, SW1 SW_SPDT

Commit message: Updated
Parts:
- added J4: FeatherWing_DCmotor, extension_circuit_board:FeatherWing_DC_Motor_Driver, F.Cu at (137.4, 88.3)
- added J5: Jetson Nano Power, extension_circuit_board:Jetson Nano Power, F.Cu at (188.0, 66.0)
- added J6: Motor Power, extension_circuit_board:Jetson Nano Power, F.Cu at (182.0, 107.0)
- added REF**: MountingHole_3.2mm_M3, MountingHole:MountingHole_3.2mm_M3, F.Cu at (192.0, 119.0)
- added REF**: MountingHole_3.2mm_M3, MountingHole:MountingHole_3.2mm_M3, F.Cu at (192.0, 53.0)
- J1: moved to B.Cu
- moved SW1 92.2 mm to (101.3, 89.0), turned to -90 degrees
- moved J1 86.8 mm to (114.3, 104.1), turned to -90 degrees
- moved J3 13.9 mm to (107.7, 63.5)
- moved J2 7.67 mm to (125.0, 63.5)
Routing:
- net I2C_2_SCL: track 20.2 -> 127.1 mm, vias 1 -> 2
- net I2C_2_SDA: track 22.9 -> 117.2 mm
- net +3.3V: track 24.2 -> 100.2 mm, vias 0 -> 1
- net +5V: track 98.8 -> 165.4 mm
- net GND: track 272.7 -> 286.8 mm
Other:
- board text added: "+5V"
- board text added: "GND"
- board text added: "Jetson Nano Power"
- board text added: "Motor Power"
- board text added: "PiOLED"
- board text added: "https://github.com/naoya1110 2023.1.4 v0.1"

Commit message: updated
Parts:
- added ?: , , F.Cu at (157.5, 114.3)
- added ?: , , F.Cu at (165.1, 114.3)
- added ?: , , F.Cu at (157.5, 116.8)
- added ?: , , F.Cu at (157.5, 111.8)
- added ?: , , F.Cu at (154.9, 116.8)
- added ?: , , F.Cu at (152.4, 111.8)
- added ?: , , F.Cu at (162.6, 111.8)
- added ?: , , F.Cu at (152.4, 114.3)
- added ?: , , F.Cu at (162.6, 114.3)
- added ?: , , F.Cu at (165.1, 111.8)
- added ?: , , F.Cu at (154.9, 114.3)
- added ?: , , F.Cu at (160.0, 111.8)
- added ?: , , F.Cu at (154.9, 119.4)
- added ?: , , F.Cu at (152.4, 116.8)
- added ?: , , F.Cu at (160.0, 114.3)
- added ?: , , F.Cu at (154.9, 111.8)
- added ?: , , F.Cu at (157.5, 119.4)
- added REF**: TestPoint_THTPad_D2.0mm_Drill1.0mm, TestPoint:TestPoint_THTPad_D2.0mm_Drill1.0mm, F.Cu at (152.4, 119.4)
Changed lines of the file:
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@@
     (tags "mounting hole 3.2mm no annular m3")
     (attr exclude_from_pos_files exclude_from_bom)
-    (fp_text reference "REF**" (at 0 -4.2) (layer "F.SilkS")
+    (fp_text reference "REF**" (at 0 -4.2) (layer "F.SilkS") hide
       (effects (font (size 1 1) (thickness 0.15)))
     )
@@
     (fp_circle (center 0 0) (end 3.45 0) (layer "F.CrtYd") (width 0.05) (fill none))
     (pad "" np_thru_hole circle (at 0 0) (size 3.2 3.2) (drill 3.2) (layers F&B.Cu *.Mask))
+  )
+  (footprint "" (layer "F.Cu")
+    (at 157.48 114.3)
+    (fp_text reference "" (at 0 0) (layer "F.SilkS")
+      (effects (font (size 1.27 1.27) (thickness 0.15)))
+    )
+    (fp_text value "" (at 0 0) (layer "F.SilkS")
+      (effects (font (size 1.27 1.27) (thickness 0.15)))
+    )
+    (pad "1" thru_hole circle (at 0 0) (size 2 2) (drill 1) (layers F&B.Cu *.Mask))
   )
   (footprint "Connector_PinHeader_2.54mm:PinHeader_2x20_P2.54mm_Vertical" (layer "F.Cu")
@@
     )
   )
+  (footprint "" (layer "F.Cu")
+    (at 165.1 111.76)
+    (fp_text reference "" (at 0 0) (layer "F.SilkS")
+      (effects (font (size 1.27 1.27) (thickness 0.15)))
+    )
+    (fp_text value "" (at 0 0) (layer "F.SilkS")
+      (effects (font (size 1.27 1.27) (thickness 0.15)))
+    )
+    (pad "1" thru_hole circle (at 0 0) (size 2 2) (drill 1) (layers F&B.Cu *.Mask))
+  )
   (footprint "extension_circuit_board:Jetson Nano Power" (layer "F.Cu")
     (at 188 66 90)
@@
     (pad "2" thru_hole circle (at 2.54 -2.54 90) (size 3 3) (drill 0.9) (layers *.Cu *.Mask)
       (net 2 "GND") (pinfunction "Pin_2") (pintype "passive"))
+  )
+  (footprint "" (layer "F.Cu")
+    (at 154.94 114.3)
+    (fp_text reference "" (at 0 0) (layer "F.SilkS")
+      (effects (font (size 1.27 1.27) (thickness 0.15)))
+    )
+    (fp_text value "" (at 0 0) (layer "F.SilkS")
+      (effects (font (size 1.27 1.27) (thickness 0.15)))
+    )
+    (pad "1" thru_hole circle (at 0 0) (size 2 2) (drill 1) (layers F&B.Cu *.Mask))
+  )
+  (footprint "" (layer "F.Cu")
+    (at 160.02 111.76)
+    (fp_text reference "" (at 0 0) (layer "F.SilkS")
+      (effects (font (size 1.27 1.27) (thickness 0.15)))
+    )
+    (fp_text value "" (at 0 0) (layer "F.SilkS")
+      (effects (font (size 1.27 1.27) (thickness 0.15)))
+    )
+    (pad "1" thru_hole circle (at 0 0) (size 2 2) (drill 1) (layers F&B.Cu *.Mask))
   )
   (footprint "MountingHole:MountingHole_3.2mm_M3" (layer "F.Cu")
@@
     (pad "4" thru_hole circle (at 0 -2.54 270) (size 2 2) (drill 0.9) (layers *.Cu *.Mask))
   )
+  (footprint "" (layer "F.Cu")
+    (at 154.94 119.38)
+    (fp_text reference "" (at 0 0) (layer "F.SilkS")
+      (effects (font (size 1.27 1.27) (thickness 0.15)))
+    )
+    (fp_text value "" (at 0 0) (layer "F.SilkS")
+      (effects (font (size 1.27 1.27) (thickness 0.15)))
+    )
+    (pad "1" thru_hole circle (at 0 0) (size 2 2) (drill 1) (layers F&B.Cu *.Mask))
+  )
+  (footprint "" (layer "F.Cu")
+    (at 152.4 116.84)
+    (fp_text reference "" (at 0 0) (layer "F.SilkS")
+      (effects (font (size 1.27 1.27) (thickness 0.15)))
+    )
+    (fp_text value "" (at 0 0) (layer "F.SilkS")
+      (effects (font (size 1.27 1.27) (thickness 0.15)))
+    )
+    (pad "1" thru_hole circle (at 0 0) (size 2 2) (drill 1) (layers F&B.Cu *.Mask))
+  )
   (footprint "MountingHole:MountingHole_3.2mm_M3" (layer "F.Cu")
     (at 103 53)
@@
     (pad "2" thru_hole circle (at 2.54 -2.54) (size 3 3) (drill 0.9) (layers *.Cu *.Mask)
       (net 2 "GND") (pinfunction "Pin_2") (pintype "passive"))
+  )
+  (footprint "" (layer "F.Cu")
+    (at 160.02 114.3)
+    (fp_text reference "" (at 0 0) (layer "F.SilkS")
+      (effects (font (size 1.27 1.27) (thickness 0.15)))
+    )
+    (fp_text value "" (at 0 0) (layer "F.SilkS")
+      (effects (font (size 1.27 1.27) (thickness 0.15)))
+    )
+    (pad "1" thru_hole circle (at 0 0) (size 2 2) (drill 1) (layers F&B.Cu *.Mask))
+  )
+  (footprint "" (layer "F.Cu")
+    (at 154.94 111.76)
+    (fp_text reference "" (at 0 0) (layer "F.SilkS")
+      (effects (font (size 1.27 1.27) (thickness 0.15)))
+    )
+    (fp_text value "" (at 0 0) (layer "F.SilkS")
+      (effects (font (size 1.27 1.27) (thickness 0.15)))
+    )
+    (pad "1" thru_hole circle (at 0 0) (size 2 2) (drill 1) (layers F&B.Cu *.Mask))
+  )
+  (footprint "" (layer "F.Cu")
+    (at 157.48 119.38)
+    (fp_text reference "" (at 0 0) (layer "F.SilkS")
+      (effects (font (size 1.27 1.27) (thickness 0.15)))
+    )
+    (fp_text value "" (at 0 0) (layer "F.SilkS")
+      (effects (font (size 1.27 1.27) (thickness 0.15)))
+    )
+    (pad "1" thru_hole circle (at 0 0) (size 2 2) (drill 1) (layers F&B.Cu *.Mask))
+  )
+  (footprint "" (layer "F.Cu")
+    (at 165.1 114.3)
+    (fp_text reference "" (at 0 0) (layer "F.SilkS")
+      (effects (font (size 1.27 1.27) (thickness 0.15)))
+    )
+    (fp_text value "" (at 0 0) (layer "F.SilkS")
+      (effects (font (size 1.27 1.27) (thickness 0.15)))
+    )
+    (pad "1" thru_hole circle (at 0 0) (size 2 2) (drill 1) (layers F&B.Cu *.Mask))
+  )
+  (footprint "TestPoint:TestPoint_THTPad_D2.0mm_Drill1.0mm" (layer "F.Cu")
+    (at 152.4 119.38)
+    (descr "THT pad as test Point, diameter 2.0mm, hole diameter 1.0mm")
+    (tags "test point THT pad")
+    (attr exclude_from_pos_files exclude_from_bom)
+    (fp_text reference "REF**" (at 0 -1.998) (layer "F.SilkS") hide
+      (effects (font (size 1 1) (thickness 0.15)))
+    )
+    (fp_text value "TestPoint_THTPad_D2.0mm_Drill1.0mm" (at 0 2.05) (layer "F.Fab")
+      (effects (font (size 1 1) (thickness 0.15)))
+    )
+    (fp_text user "${REFERENCE}" (at 0 -2) (layer "F.Fab")
+      (effects (font (size 1 1) (thickness 0.15)))
+    )
+    (fp_circle (center 0 0) (end 0 1.2) (layer "F.SilkS") (width 0.12) (fill none))
+    (fp_circle (center 0 0) (end 1.5 0) (layer "F.CrtYd") (width 0.05) (fill none))
+    (pad "1" thru_hole circle (at 0 0) (size 2 2) (drill 1) (layers *.Cu *.Mask))
+  )
+  (footprint "" (layer "F.Cu")
+    (at 157.48 116.84)
+    (fp_text reference "" (at 0 0) (layer "F.SilkS")
+      (effects (font (size 1.27 1.27) (thickness 0.15)))
+    )
+    (fp_text value "" (at 0 0) (layer "F.SilkS")
+      (effects (font (size 1.27 1.27) (thickness 0.15)))
+    )
+    (pad "1" thru_hole circle (at 0 0) (size 2 2) (drill 1) (layers F&B.Cu *.Mask))
+  )
+  (footprint "" (layer "F.Cu")
+    (at 157.48 111.76)
+    (fp_text reference "" (at 0 0) (layer "F.SilkS")
+      (effects (font (size 1.27 1.27) (thickness 0.15)))
+    )
+    (fp_text value "" (at 0 0) (layer "F.SilkS")
+      (effects (font (size 1.27 1.27) (thickness 0.15)))
+    )
+    (pad "1" thru_hole circle (at 0 0) (size 2 2) (drill 1) (layers F&B.Cu *.Mask))
+  )
+  (footprint "" (layer "F.Cu")
+    (at 154.94 116.84)
+    (fp_text reference "" (at 0 0) (layer "F.SilkS")
+      (effects (font (size 1.27 1.27) (thickness 0.15)))
+    )
+    (fp_text value "" (at 0 0) (layer "F.SilkS")
+      (effects (font (size 1.27 1.27) (thickness 0.15)))
+    )
+    (pad "1" thru_hole circle (at 0 0) (size 2 2) (drill 1) (layers F&B.Cu *.Mask))
+  )
+  (footprint "" (layer "F.Cu")
+    (at 152.4 111.76)
+    (fp_text reference "" (at 0 0) (layer "F.SilkS")
+      (effects (font (size 1.27 1.27) (thickness 0.15)))
+    )
+    (fp_text value "" (at 0 0) (layer "F.SilkS")
+      (effects (font (size 1.27 1.27) (thickness 0.15)))
+    )
+    (pad "1" thru_hole circle (at 0 0) (size 2 2) (drill 1) (layers F&B.Cu *.Mask))
   )
   (footprint "extension_circuit_board:FeatherWing_DC_Motor_Driver" (layer "F.Cu")
@@
       (net 29 "I2C_2_SDA") (pinfunction "Pin_32") (pintype "passive"))
   )
+  (footprint "" (layer "F.Cu")
+    (at 162.56 111.76)
+    (fp_text reference "" (at 0 0) (layer "F.SilkS")
+      (effects (font (size 1.27 1.27) (thickness 0.15)))
+    )
+    (fp_text value "" (at 0 0) (layer "F.SilkS")
+      (effects (font (size 1.27 1.27) (thickness 0.15)))
+    )
+    (pad "1" thru_hole circle (at 0 0) (size 2 2) (drill 1) (layers F&B.Cu *.Mask))
+  )
   (footprint "Connector_PinHeader_2.54mm:PinHeader_2x03_P2.54mm_Vertical" (layer "F.Cu")
     (at 107.725 63.475)
@@
     (pad "" np_thru_hole circle (at 0 0) (size 3.2 3.2) (drill 3.2) (layers F&B.Cu *.Mask))
   )
+  (footprint "" (layer "F.Cu")
+    (at 152.4 114.3)
+    (fp_text reference "" (at 0 0) (layer "F.SilkS")
+      (effects (font (size 1.27 1.27) (thickness 0.15)))
+    )
+    (fp_text value "" (at 0 0) (layer "F.SilkS")
+      (effects (font (size 1.27 1.27) (thickness 0.15)))
+    )
+    (pad "1" thru_hole circle (at 0 0) (size 2 2) (drill 1) (layers F&B.Cu *.Mask))
+  )
+  (footprint "" (layer "F.Cu")
+    (at 162.56 114.3)
+    (fp_text reference "" (at 0 0) (layer "F.SilkS")
+      (effects (font (size 1.27 1.27) (thickness 0.15)))
+    )
+    (fp_text value "" (at 0 0) (layer "F.SilkS")
+      (effects (font (size 1.27 1.27) (thickness 0.15)))
+    )
+    (pad "1" thru_hole circle (at 0 0) (size 2 2) (drill 1) (layers F&B.Cu *.Mask))
+  )
   (footprint "extension_circuit_board:AE_MRUSB_DIP" (layer "B.Cu")
     (at 114.3 104.14 -90)
@@
     (effects (font (size 1 1) (thickness 0.15)))
   )
-  (gr_text "https://github.com/naoya1110\n2023.1.4 v0.1" (at 157.5 117.5) (layer "F.SilkS")
+  (gr_text "https://github.com/naoya1110\n2023.1.4 v0.1" (at 162.56 117.5) (layer "F.SilkS")
     (effects (font (size 1 1) (thickness 0.15)) (justify left))
   )

Commit message: updated
Parts:
- removed ? (x17): , 
- removed the REF** at (192.0, 119.0)
- removed the REF** at (103.0, 119.0)
- removed the REF** at (103.0, 53.0)
- removed the REF** at (152.4, 119.4)
- removed the REF** at (192.0, 53.0)
- added J7: GPIO_odd, Connector_PinHeader_2.54mm:PinHeader_1x20_P2.54mm_Vertical, F.Cu at (141.2, 60.6)
- added J8: GPIO_even, Connector_PinHeader_2.54mm:PinHeader_1x20_P2.54mm_Vertical, F.Cu at (152.2, 60.6)
- added REF**: MountingHole_3.2mm_M3, MountingHole:MountingHole_3.2mm_M3, F.Cu at (213.0, 50.0)
- added REF**: MountingHole_3.2mm_M3, MountingHole:MountingHole_3.2mm_M3, F.Cu at (124.0, 50.0)
- added REF**: MountingHole_3.2mm_M3, MountingHole:MountingHole_3.2mm_M3, F.Cu at (124.0, 116.0)
- added REF**: MountingHole_3.2mm_M3, MountingHole:MountingHole_3.2mm_M3, F.Cu at (213.0, 116.0)
- moved SW1 21.5 mm to (122.4, 92.7)
- moved J3 21.4 mm to (128.9, 60.6)
- moved J6 21.0 mm to (202.9, 104.7)
- moved J5 20.9 mm to (208.8, 64.1)
- moved J2 20.6 mm to (145.4, 60.6)
- moved J4 20.0 mm to (157.4, 87.3)
- moved J1 19.6 mm to (133.8, 103.8)
Connections:
- J2 pad 10: unconnected-(J2-Pad10) -> Net-(J2-Pad10)
- J2 pad 11: unconnected-(J2-Pad11) -> Net-(J2-Pad11)
- J2 pad 12: unconnected-(J2-Pad12) -> Net-(J2-Pad12)
- J2 pad 13: unconnected-(J2-Pad13) -> Net-(J2-Pad13)
- J2 pad 15: unconnected-(J2-Pad15) -> Net-(J2-Pad15)
- J2 pad 16: unconnected-(J2-Pad16) -> Net-(J2-Pad16)
- J2 pad 17: unconnected-(J2-Pad17) -> Net-(J2-Pad17)
- J2 pad 18: unconnected-(J2-Pad18) -> Net-(J2-Pad18)
- J2 pad 19: unconnected-(J2-Pad19) -> Net-(J2-Pad19)
- J2 pad 21: unconnected-(J2-Pad21) -> Net-(J2-Pad21)
- J2 pad 22: unconnected-(J2-Pad22) -> Net-(J2-Pad22)
- J2 pad 23: unconnected-(J2-Pad23) -> Net-(J2-Pad23)
- J2 pad 24: unconnected-(J2-Pad24) -> Net-(J2-Pad24)
- J2 pad 26: unconnected-(J2-Pad26) -> Net-(J2-Pad26)
- J2 pad 27: unconnected-(J2-Pad27) -> Net-(J2-Pad27)
- J2 pad 28: unconnected-(J2-Pad28) -> Net-(J2-Pad28)
- J2 pad 29: unconnected-(J2-Pad29) -> Net-(J2-Pad29)
- J2 pad 31: unconnected-(J2-Pad31) -> Net-(J2-Pad31)
- J2 pad 32: unconnected-(J2-Pad32) -> Net-(J2-Pad32)
- J2 pad 33: unconnected-(J2-Pad33) -> Net-(J2-Pad33)
- J2 pad 35: unconnected-(J2-Pad35) -> Net-(J2-Pad35)
- J2 pad 36: unconnected-(J2-Pad36) -> Net-(J2-Pad36)
- J2 pad 37: unconnected-(J2-Pad37) -> Net-(J2-Pad37)
- J2 pad 38: unconnected-(J2-Pad38) -> Net-(J2-Pad38)
- J2 pad 40: unconnected-(J2-Pad40) -> Net-(J2-Pad40)
- J2 pad 7: unconnected-(J2-Pad7) -> Net-(J2-Pad7)
- J2 pad 8: unconnected-(J2-Pad8) -> Net-(J2-Pad8)
Routing:
- net I2C_2_SCL: track 127.1 -> 111.8 mm, vias 2 -> 1
- net +5V: track 165.4 -> 172.1 mm
- net GND: track 286.8 -> 293.3 mm
- net I2C_2_SDA: track 117.2 -> 122.0 mm, vias 1 -> 2
- net Net-(J1-Pad3): track 19.6 -> 14.9 mm
- net Net-(J2-Pad8): track 0.00 -> 4.26 mm
- net Net-(J2-Pad40): track 0.00 -> 4.26 mm
- net Net-(J2-Pad38): track 0.00 -> 4.26 mm
- net Net-(J2-Pad36): track 0.00 -> 4.26 mm
- net Net-(J2-Pad32): track 0.00 -> 4.26 mm
- net Net-(J2-Pad28): track 0.00 -> 4.26 mm
- net Net-(J2-Pad26): track 0.00 -> 4.26 mm
- net Net-(J2-Pad24): track 0.00 -> 4.26 mm
- net Net-(J2-Pad22): track 0.00 -> 4.26 mm
- net Net-(J2-Pad18): track 0.00 -> 4.26 mm
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Other:
- board text removed: "+5V"
- board text removed: "GND"
- board text removed: "Jetson Nano Power"
- board text removed: "Motor Power"
- board text removed: "PiOLED"
- board text removed: "https://github.com/naoya1110 2023.1.4 v0.1"

Commit message: updated
Parts:
- added ?: , , F.Cu at (203.2, 53.3)
- added ?: , , F.Cu at (170.2, 61.0)
- added ?: , , F.Cu at (200.7, 55.9)
- added ?: , , F.Cu at (205.7, 111.8)
- added ?: , , F.Cu at (182.9, 114.3)
- added ?: , , F.Cu at (188.0, 63.5)
- added ?: , , F.Cu at (193.0, 58.4)
- added ?: , , F.Cu at (177.8, 111.8)
- added ?: , , F.Cu at (188.0, 114.3)
- added ?: , , F.Cu at (165.1, 53.3)
- added ?: , , F.Cu at (170.2, 106.7)
- added ?: , , F.Cu at (198.1, 50.8)
- added ?: , , F.Cu at (172.7, 63.5)
- added ?: , , F.Cu at (198.1, 66.0)
- added ?: , , F.Cu at (182.9, 63.5)
- added ?: , , F.Cu at (190.5, 111.8)
- added ?: , , F.Cu at (195.6, 68.6)
- added ?: , , F.Cu at (172.7, 50.8)
- added ?: , , F.Cu at (180.3, 55.9)
- added ?: , , F.Cu at (193.0, 53.3)
- added ?: , , F.Cu at (167.6, 55.9)
- added ?: , , F.Cu at (190.5, 104.1)
- added ?: , , F.Cu at (175.3, 55.9)
- added ?: , , F.Cu at (165.1, 63.5)
- added ?: , , F.Cu at (200.7, 109.2)
- added ?: , , F.Cu at (177.8, 66.0)
- added ?: , , F.Cu at (177.8, 68.6)
- added ?: , , F.Cu at (180.3, 109.2)
- added ?: , , F.Cu at (203.2, 109.2)
- added ?: , , F.Cu at (200.7, 53.3)
- added ?: , , F.Cu at (195.6, 114.3)
- added ?: , , F.Cu at (205.7, 114.3)
- added ?: , , F.Cu at (198.1, 109.2)
- added ?: , , F.Cu at (170.2, 50.8)
- added ?: , , F.Cu at (198.1, 114.3)
- added ?: , , F.Cu at (167.6, 68.6)
- added ?: , , F.Cu at (195.6, 111.8)
- added ?: , , F.Cu at (177.8, 50.8)
- added ?: , , F.Cu at (195.6, 106.7)
- added ?: , , F.Cu at (193.0, 66.0)
- added ?: , , F.Cu at (203.2, 114.3)
- added ?: , , F.Cu at (177.8, 63.5)
- added ?: , , F.Cu at (182.9, 53.3)
- added ?: , , F.Cu at (182.9, 55.9)
- added ?: , , F.Cu at (165.1, 55.9)
- added ?: , , F.Cu at (175.3, 50.8)
- added ?: , , F.Cu at (175.3, 114.3)
- added ?: , , F.Cu at (198.1, 68.6)
- added ?: , , F.Cu at (193.0, 68.6)
- added ?: , , F.Cu at (185.4, 104.1)
- added ?: , , F.Cu at (200.7, 50.8)
- added ?: , , F.Cu at (170.2, 66.0)
- added ?: , , F.Cu at (185.4, 53.3)
- added ?: , , F.Cu at (190.5, 66.0)
- added ?: , , F.Cu at (175.3, 58.4)
- added ?: , , F.Cu at (182.9, 61.0)
- added ?: , , F.Cu at (188.0, 61.0)
- added ?: , , F.Cu at (190.5, 53.3)
- added ?: , , F.Cu at (185.4, 50.8)
- added ?: , , F.Cu at (180.3, 104.1)
- added ?: , , F.Cu at (185.4, 109.2)
- added ?: , , F.Cu at (200.7, 63.5)
- added ?: , , F.Cu at (195.6, 109.2)
- added ?: , , F.Cu at (167.6, 114.3)
- added ?: , , F.Cu at (162.6, 111.8)
- added ?: , , F.Cu at (193.0, 104.1)
- added ?: , , F.Cu at (177.8, 114.3)
- added ?: , , F.Cu at (182.9, 109.2)
- added ?: , , F.Cu at (162.6, 53.3)
- added ?: , , F.Cu at (182.9, 66.0)
- added ?: , , F.Cu at (195.6, 61.0)
- added ?: , , F.Cu at (162.6, 50.8)
- added ?: , , F.Cu at (200.7, 68.6)
- added ?: , , F.Cu at (165.1, 50.8)
- added ?: , , F.Cu at (182.9, 106.7)
- added ?: , , F.Cu at (188.0, 58.4)
- added ?: , , F.Cu at (185.4, 61.0)
- added ?: , , F.Cu at (198.1, 53.3)
- added ?: , , F.Cu at (172.7, 66.0)
- added ?: , , F.Cu at (185.4, 68.6)
- added ?: , , F.Cu at (180.3, 106.7)
- added ?: , , F.Cu at (180.3, 50.8)
- added ?: , , F.Cu at (193.0, 50.8)
- added ?: , , F.Cu at (190.5, 50.8)
- added ?: , , F.Cu at (165.1, 68.6)
- added ?: , , F.Cu at (182.9, 68.6)
- added ?: , , F.Cu at (190.5, 55.9)
- added ?: , , F.Cu at (167.6, 66.0)
- added ?: , , F.Cu at (200.7, 66.0)
- added ?: , , F.Cu at (180.3, 53.3)
- added ?: , , F.Cu at (177.8, 55.9)
- added ?: , , F.Cu at (200.7, 58.4)
- added ?: , , F.Cu at (167.6, 111.8)
- added ?: , , F.Cu at (195.6, 66.0)
- added ?: , , F.Cu at (170.2, 53.3)
- added ?: , , F.Cu at (170.2, 104.1)
- added ?: , , F.Cu at (180.3, 111.8)
- added ?: , , F.Cu at (188.0, 55.9)
- added ?: , , F.Cu at (180.3, 66.0)
- added ?: , , F.Cu at (177.8, 106.7)
- added ?: , , F.Cu at (203.2, 111.8)
- added ?: , , F.Cu at (167.6, 58.4)
- added ?: , , F.Cu at (193.0, 109.2)
- added ?: , , F.Cu at (185.4, 114.3)
- added ?: , , F.Cu at (170.2, 111.8)
- added ?: , , F.Cu at (177.8, 53.3)
- added ?: , , F.Cu at (193.0, 106.7)
- added ?: , , F.Cu at (175.3, 63.5)
- added ?: , , F.Cu at (172.7, 53.3)
- added ?: , , F.Cu at (167.6, 63.5)
- added ?: , , F.Cu at (195.6, 53.3)
- added ?: , , F.Cu at (200.7, 114.3)
- added ?: , , F.Cu at (188.0, 104.1)
- added ?: , , F.Cu at (190.5, 114.3)
- added ?: , , F.Cu at (195.6, 63.5)
- added ?: , , F.Cu at (175.3, 104.1)
- added ?: , , F.Cu at (188.0, 50.8)
- added ?: , , F.Cu at (177.8, 109.2)
- added ?: , , F.Cu at (172.7, 68.6)
- added ?: , , F.Cu at (193.0, 111.8)
- added ?: , , F.Cu at (188.0, 68.6)
- added ?: , , F.Cu at (170.2, 114.3)
- added ?: , , F.Cu at (177.8, 104.1)
- added ?: , , F.Cu at (198.1, 61.0)
- added ?: , , F.Cu at (162.6, 114.3)
- added ?: , , F.Cu at (177.8, 61.0)
- added ?: , , F.Cu at (175.3, 53.3)
- added ?: , , F.Cu at (180.3, 63.5)
- added ?: , , F.Cu at (190.5, 61.0)
- added ?: , , F.Cu at (190.5, 106.7)
- added ?: , , F.Cu at (162.6, 55.9)
- added ?: , , F.Cu at (172.7, 55.9)
- added ?: , , F.Cu at (188.0, 109.2)
- added ?: , , F.Cu at (203.2, 50.8)
- added ?: , , F.Cu at (170.2, 68.6)
- added ?: , , F.Cu at (170.2, 58.4)
- added ?: , , F.Cu at (175.3, 111.8)
- added ?: , , F.Cu at (167.6, 50.8)
- added ?: , , F.Cu at (193.0, 114.3)
- added ?: , , F.Cu at (165.1, 114.3)
- added ?: , , F.Cu at (188.0, 111.8)
- added ?: , , F.Cu at (185.4, 55.9)
- added ?: , , F.Cu at (172.7, 109.2)
- added ?: , , F.Cu at (198.1, 63.5)
- added ?: , , F.Cu at (170.2, 109.2)
- added ?: , , F.Cu at (182.9, 50.8)
- added ?: , , F.Cu at (195.6, 50.8)
- added ?: , , F.Cu at (200.7, 111.8)
- added ?: , , F.Cu at (175.3, 61.0)
- added ?: , , F.Cu at (165.1, 106.7)
- added ?: , , F.Cu at (165.1, 58.4)
- added ?: , , F.Cu at (172.7, 106.7)
- added ?: , , F.Cu at (193.0, 55.9)
- added ?: , , F.Cu at (162.6, 106.7)
- added ?: , , F.Cu at (167.6, 106.7)
- added ?: , , F.Cu at (195.6, 55.9)
- added ?: , , F.Cu at (180.3, 68.6)
- added ?: , , F.Cu at (185.4, 58.4)
- added ?: , , F.Cu at (198.1, 55.9)
- added ?: , , F.Cu at (180.3, 114.3)
- added ?: , , F.Cu at (188.0, 106.7)
- added ?: , , F.Cu at (198.1, 111.8)
- added ?: , , F.Cu at (177.8, 58.4)
- added ?: , , F.Cu at (185.4, 66.0)
- added ?: , , F.Cu at (203.2, 55.9)
- added ?: , , F.Cu at (180.3, 61.0)
- added ?: , , F.Cu at (172.7, 104.1)
- added ?: , , F.Cu at (200.7, 61.0)
- added ?: , , F.Cu at (175.3, 68.6)
- added ?: , , F.Cu at (172.7, 114.3)
- added ?: , , F.Cu at (185.4, 111.8)
- added ?: , , F.Cu at (165.1, 66.0)
- added ?: , , F.Cu at (170.2, 63.5)
- added ?: , , F.Cu at (190.5, 109.2)
- added ?: , , F.Cu at (190.5, 68.6)
- added ?: , , F.Cu at (167.6, 61.0)
- added ?: , , F.Cu at (182.9, 104.1)
- added ?: , , F.Cu at (170.2, 55.9)
- added ?: , , F.Cu at (167.6, 109.2)
- added ?: , , F.Cu at (172.7, 58.4)
- added ?: , , F.Cu at (172.7, 111.8)
- added ?: , , F.Cu at (198.1, 58.4)
- added ?: , , F.Cu at (162.6, 61.0)
- added ?: , , F.Cu at (190.5, 63.5)
- added ?: , , F.Cu at (182.9, 111.8)
- added ?: , , F.Cu at (195.6, 58.4)
- added ?: , , F.Cu at (180.3, 58.4)
- added ?: , , F.Cu at (165.1, 61.0)
- added ?: , , F.Cu at (190.5, 58.4)
- added ?: , , F.Cu at (188.0, 53.3)
- added ?: , , F.Cu at (188.0, 66.0)
- added ?: , , F.Cu at (162.6, 58.4)
- added ?: , , F.Cu at (175.3, 109.2)
- added ?: , , F.Cu at (162.6, 109.2)
- added ?: , , F.Cu at (193.0, 63.5)
- added ?: , , F.Cu at (182.9, 58.4)
- added ?: , , F.Cu at (193.0, 61.0)
- added ?: , , F.Cu at (185.4, 106.7)
- added ?: , , F.Cu at (205.7, 109.2)
- added ?: , , F.Cu at (175.3, 106.7)
- added ?: , , F.Cu at (172.7, 61.0)
- added ?: , , F.Cu at (165.1, 111.8)
- added ?: , , F.Cu at (185.4, 63.5)
- added ?: , , F.Cu at (165.1, 109.2)
- added ?: , , F.Cu at (167.6, 53.3)
- added ?: , , F.Cu at (175.3, 66.0)
Routing:
- net +5V: track 172.1 -> 116.5 mm
- net +3.3V: track 101.6 -> 111.8 mm, vias 2 -> 3
Other:
- board text added: "J6"

Commit message: updated
Parts:
- added ?: , , F.Cu at (205.7, 50.8)
- added ?: , , F.Cu at (205.7, 55.9)
- added ?: , , F.Cu at (205.7, 53.3)
Connections:
- J2 pad 17: Net-(J2-Pad17) -> +3.3V
- J7 pad 9: Net-(J2-Pad17) -> +3.3V
Routing:
- net +3.3V: track 111.8 -> 136.9 mm, vias 3 -> 5
- net Net-(J2-Pad17): track 4.20 -> 0.00 mm
- net GND: track 293.3 -> 291.5 mm
- net +5V: track 116.5 -> 115.0 mm
- net I2C_2_SDA: track 122.0 -> 123.3 mm
- net I2C_2_SCL: track 111.8 -> 112.5 mm
Other:
- board text added: "+3.3V"
- board text added: "+5V"
- board text added: "10"
- board text added: "11"
- board text added: "12"
- board text added: "13"
- board text added: "15"
- board text added: "16"
- board text added: "18"
- board text added: "19"
- board text added: "21"
- board text added: "22"
- board text added: "23"
- board text added: "24"
- board text added: "26"
- board text added: "27"
- board text added: "28"
- board text added: "29"
- board text added: "31"
- board text added: "32"
- board text added: "33"
- board text added: "35"
- board text added: "36"
- board text added: "37"
- board text added: "38"
- board text added: "40"
- board text added: "7"
- board text added: "8"
- board text added: "AE_MRUSB_DIP"
- board text added: "FeatherWing DC Motor Driver"
- board text added: "GND"
- board text added: "JetBot Extension Board v.0.1 2023 Jan. https://github.com/naoya1110/jetbot_3d_model"
- board text added: "Jetson Nano Power"
- board text added: "Motor Power"
- board text added: "POWER SW"
- board text added: "PiOLED"
- board text added: "SCL"
- board text added: "SDA"
