File: extension_circuit_board/extension_circuit_board.kicad_pcb (KiCad board)
At the start: 2 copper layers, 95 x 72 mm, 222 parts, among them J1 AE_MRUSB_DIP, J2 Jetson_Nano_GPIO, J3 PiOLED 2x3, J4 FeatherWing_DCmotor, J5 Jetson Nano Power, J6 Motor Power, J7 GPIO_odd, J8 GPIO_even, SW1 SW_SPDT

Commit message: Updated
Parts:
- added ?: , , F.Cu at (162.6, 63.5)
- added ?: , , F.Cu at (162.6, 68.6)
- added ?: , , F.Cu at (162.6, 66.0)
Changed lines of the file:
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@@
+  )
+  (footprint "" (layer "F.Cu")
+    (at 162.56 68.58)
+    (fp_text reference "" (at 0 0) (layer "F.SilkS")
+      (effects (font (size 1.27 1.27) (thickness 0.15)))
+    )
+    (fp_text value "" (at 0 0) (layer "F.SilkS")
+      (effects (font (size 1.27 1.27) (thickness 0.15)))
+    )
+    (pad "1" thru_hole circle (at 0 0) (size 2 2) (drill 1) (layers F&B.Cu *.Mask))
   )
   (footprint "" (layer "F.Cu")
@@
   (footprint "" (layer "F.Cu")
     (at 185.42 63.5)
+    (fp_text reference "" (at 0 0) (layer "F.SilkS")
+      (effects (font (size 1.27 1.27) (thickness 0.15)))
+    )
+    (fp_text value "" (at 0 0) (layer "F.SilkS")
+      (effects (font (size 1.27 1.27) (thickness 0.15)))
+    )
+    (pad "1" thru_hole circle (at 0 0) (size 2 2) (drill 1) (layers F&B.Cu *.Mask))
+  )
+  (footprint "" (layer "F.Cu")
+    (at 162.56 66.04)
     (fp_text reference "" (at 0 0) (layer "F.SilkS")
       (effects (font (size 1.27 1.27) (thickness 0.15)))
@@
     (fp_text reference "" (at 0 0) (layer "F.SilkS")
       (effects (font (size 1.27 1.27) (thickness 0.15)))
+    )
+    (fp_text value "" (at 0 0) (layer "F.SilkS")
+      (effects (font (size 1.27 1.27) (thickness 0.15)))
+    )
+    (pad "1" thru_hole circle (at 0 0) (size 2 2) (drill 1) (layers F&B.Cu *.Mask))
+  )
+  (footprint "" (layer "F.Cu")
+    (at 162.56 63.5)
+    (fp_text reference "" (at 0 0) (layer "F.SilkS")
+      (effects (font (size 1.27 1.27) (thickness 0.15)))
