File: extension_circuit_board/v2/extension_circuit_board.kicad_pcb (KiCad board)
At the start: 2 copper layers, 95 x 72 mm, 13 parts, among them J1 GPIO_odd, J2 Jetson_Nano_GPIO, J3 GPIO_even, J4 FeatherWing_DCmotor, J5 PiOLED 2x3, J6 Motor Power, J7 Battery In, SW1 SW_SPDT, U1 DFR0753

Commit message: updated
Parts:
- added ?: , , F.Cu at (205.7, 106.7)
- added ?: , , F.Cu at (195.6, 106.7)
- added ?: , , F.Cu at (200.7, 114.3)
- added ?: , , F.Cu at (177.8, 53.3)
- added ?: , , F.Cu at (165.1, 50.8)
- added ?: , , F.Cu at (180.3, 50.8)
- added ?: , , F.Cu at (193.0, 104.1)
- added ?: , , F.Cu at (172.7, 50.8)
- added ?: , , F.Cu at (210.8, 109.2)
- added ?: , , F.Cu at (198.1, 111.8)
- added ?: , , F.Cu at (198.1, 109.2)
- added ?: , , F.Cu at (160.0, 53.3)
- added ?: , , F.Cu at (203.2, 111.8)
- added ?: , , F.Cu at (208.3, 91.4)
- added ?: , , F.Cu at (205.7, 111.8)
- added ?: , , F.Cu at (210.8, 104.1)
- added ?: , , F.Cu at (203.2, 106.7)
- added ?: , , F.Cu at (190.5, 50.8)
- added ?: , , F.Cu at (177.8, 50.8)
- added ?: , , F.Cu at (208.3, 101.6)
- added ?: , , F.Cu at (205.7, 114.3)
- added ?: , , F.Cu at (160.0, 50.8)
- added ?: , , F.Cu at (167.6, 50.8)
- added ?: , , F.Cu at (193.0, 53.3)
- added ?: , , F.Cu at (182.9, 53.3)
- added ?: , , F.Cu at (188.0, 53.3)
- added ?: , , F.Cu at (165.1, 53.3)
- added ?: , , F.Cu at (193.0, 106.7)
- added ?: , , F.Cu at (205.7, 104.1)
- added ?: , , F.Cu at (195.6, 104.1)
- added ?: , , F.Cu at (170.2, 53.3)
- added ?: , , F.Cu at (200.7, 106.7)
- added ?: , , F.Cu at (193.0, 109.2)
- added ?: , , F.Cu at (198.1, 106.7)
- added ?: , , F.Cu at (195.6, 111.8)
- added ?: , , F.Cu at (203.2, 114.3)
- added ?: , , F.Cu at (200.7, 104.1)
- added ?: , , F.Cu at (167.6, 53.3)
- added ?: , , F.Cu at (198.1, 114.3)
- added ?: , , F.Cu at (195.6, 114.3)
- added ?: , , F.Cu at (185.4, 50.8)
- added ?: , , F.Cu at (210.8, 88.9)
- added ?: , , F.Cu at (210.8, 94.0)
- added ?: , , F.Cu at (208.3, 99.1)
- added ?: , , F.Cu at (208.3, 96.5)
- added ?: , , F.Cu at (208.3, 104.1)
- added ?: , , F.Cu at (185.4, 53.3)
- added ?: , , F.Cu at (188.0, 50.8)
- added ?: , , F.Cu at (193.0, 111.8)
- added ?: , , F.Cu at (210.8, 86.4)
- added ?: , , F.Cu at (198.1, 104.1)
- added ?: , , F.Cu at (205.7, 101.6)
- added ?: , , F.Cu at (200.7, 109.2)
- added ?: , , F.Cu at (182.9, 50.8)
- added ?: , , F.Cu at (208.3, 94.0)
- added ?: , , F.Cu at (203.2, 109.2)
- added ?: , , F.Cu at (205.7, 109.2)
- added ?: , , F.Cu at (162.6, 53.3)
- added ?: , , F.Cu at (208.3, 111.8)
- added ?: , , F.Cu at (190.5, 53.3)
- added ?: , , F.Cu at (210.8, 91.4)
- added ?: , , F.Cu at (175.3, 53.3)
- added ?: , , F.Cu at (208.3, 109.2)
- added ?: , , F.Cu at (208.3, 106.7)
- added ?: , , F.Cu at (200.7, 111.8)
- added ?: , , F.Cu at (193.0, 114.3)
- added ?: , , F.Cu at (210.8, 96.5)
- added ?: , , F.Cu at (180.3, 53.3)
- added ?: , , F.Cu at (208.3, 86.4)
- added ?: , , F.Cu at (210.8, 106.7)
- added ?: , , F.Cu at (175.3, 50.8)
- added ?: , , F.Cu at (172.7, 53.3)
- added ?: , , F.Cu at (170.2, 50.8)
- added ?: , , F.Cu at (208.3, 88.9)
- added ?: , , F.Cu at (210.8, 101.6)
- added ?: , , F.Cu at (162.6, 50.8)
- added ?: , , F.Cu at (203.2, 104.1)
- added ?: , , F.Cu at (193.0, 50.8)
- added ?: , , F.Cu at (210.8, 99.1)
- added ?: , , F.Cu at (195.6, 109.2)
Routing:
- net GND: track 274.6 -> 279.5 mm
- net +9V: track 29.7 -> 31.5 mm
- added copper zone on F.Cu, net +5V
- added copper zone on B.Cu, net GND
Other:
- board text added: "JetBot Extension Board v.2 2024 Jun. https://github.com/naoya1110/jetbot_3d_model"
- board text removed: "JetBot Extension Board v.2 2025 Jun. https://github.com/naoya1110/jetbot_3d_model"

Commit message: Updated
Parts:
- removed ? (x80): , 
- added J8: I2C 2x3, Connector_PinHeader_2.54mm:PinHeader_2x03_P2.54mm_Vertical, F.Cu at (128.5, 86.0)
- J1: renamed from J7; value Battery In -> Battery
- moved SW1 93.3 mm to (215.2, 103.0), turned to 90 degrees
- moved J1 14.5 mm to (212.5, 92.5), turned to 90 degrees
- renumbered J6 to J2, J1 to J3, J2 to J4, J3 to J5, J4 to J6, J5 to J7
Connections:
- J1 pad 1: +9V -> Net-(SW1-Pad1)
- SW1 pad 2: +5V -> +9V
- U1 pad 4: Net-(SW1-Pad1) -> +5V
Routing:
- net Net-(SW1-Pad1): track 112.3 -> 0.00 mm
- net GND: track 279.5 -> 226.3 mm, vias 2 -> 0
- net +5V: track 88.7 -> 41.7 mm
- net +3.3V: track 108.9 -> 70.3 mm, vias 4 -> 1
- net I2C_2_SDA: track 73.5 -> 41.8 mm
- net +9V: track 31.5 -> 0.00 mm
- net I2C_2_SCL: track 71.7 -> 44.1 mm, vias 2 -> 1
- removed copper zone on F.Cu, net +5V
- removed copper zone on B.Cu, net GND
Other:
- board text added: "JetBot Extension Board v.2.1 2024 Jun. https://github.com/naoya1110/jetbot_3d_model"
- board text removed: "JetBot Extension Board v.2 2024 Jun. https://github.com/naoya1110/jetbot_3d_model"

Commit message: updated
Parts:
- added REF**: TestPoint_THTPad_D1.5mm_Drill0.7mm, TestPoint:TestPoint_THTPad_D1.5mm_Drill0.7mm, F.Cu at (205.7, 106.7)
- added REF**: TestPoint_THTPad_D1.5mm_Drill0.7mm, TestPoint:TestPoint_THTPad_D1.5mm_Drill0.7mm, F.Cu at (157.5, 53.3)
- added REF**: TestPoint_THTPad_D1.5mm_Drill0.7mm, TestPoint:TestPoint_THTPad_D1.5mm_Drill0.7mm, F.Cu at (198.1, 111.8)
- added REF**: TestPoint_THTPad_D1.5mm_Drill0.7mm, TestPoint:TestPoint_THTPad_D1.5mm_Drill0.7mm, F.Cu at (154.9, 53.3)
- added REF**: TestPoint_THTPad_D1.5mm_Drill0.7mm, TestPoint:TestPoint_THTPad_D1.5mm_Drill0.7mm, F.Cu at (200.7, 111.8)
- added REF**: TestPoint_THTPad_D1.5mm_Drill0.7mm, TestPoint:TestPoint_THTPad_D1.5mm_Drill0.7mm, F.Cu at (198.1, 106.7)
- added REF**: TestPoint_THTPad_D1.5mm_Drill0.7mm, TestPoint:TestPoint_THTPad_D1.5mm_Drill0.7mm, F.Cu at (205.7, 109.2)
- added REF**: TestPoint_THTPad_D1.5mm_Drill0.7mm, TestPoint:TestPoint_THTPad_D1.5mm_Drill0.7mm, F.Cu at (203.2, 104.1)
- added REF**: TestPoint_THTPad_D1.5mm_Drill0.7mm, TestPoint:TestPoint_THTPad_D1.5mm_Drill0.7mm, F.Cu at (180.3, 50.8)
- added REF**: TestPoint_THTPad_D1.5mm_Drill0.7mm, TestPoint:TestPoint_THTPad_D1.5mm_Drill0.7mm, F.Cu at (195.6, 101.6)
- added REF**: TestPoint_THTPad_D1.5mm_Drill0.7mm, TestPoint:TestPoint_THTPad_D1.5mm_Drill0.7mm, F.Cu at (203.2, 114.3)
- added REF**: TestPoint_THTPad_D1.5mm_Drill0.7mm, TestPoint:TestPoint_THTPad_D1.5mm_Drill0.7mm, F.Cu at (182.9, 50.8)
- added REF**: TestPoint_THTPad_D1.5mm_Drill0.7mm, TestPoint:TestPoint_THTPad_D1.5mm_Drill0.7mm, F.Cu at (200.7, 53.3)
- added REF**: TestPoint_THTPad_D1.5mm_Drill0.7mm, TestPoint:TestPoint_THTPad_D1.5mm_Drill0.7mm, F.Cu at (137.2, 53.3)
- added REF**: TestPoint_THTPad_D1.5mm_Drill0.7mm, TestPoint:TestPoint_THTPad_D1.5mm_Drill0.7mm, F.Cu at (182.9, 53.3)
- added REF**: TestPoint_THTPad_D1.5mm_Drill0.7mm, TestPoint:TestPoint_THTPad_D1.5mm_Drill0.7mm, F.Cu at (193.0, 114.3)
- added REF**: TestPoint_THTPad_D1.5mm_Drill0.7mm, TestPoint:TestPoint_THTPad_D1.5mm_Drill0.7mm, F.Cu at (200.7, 109.2)
- added REF**: TestPoint_THTPad_D1.5mm_Drill0.7mm, TestPoint:TestPoint_THTPad_D1.5mm_Drill0.7mm, F.Cu at (170.2, 53.3)
- added REF**: TestPoint_THTPad_D1.5mm_Drill0.7mm, TestPoint:TestPoint_THTPad_D1.5mm_Drill0.7mm, F.Cu at (213.4, 104.1)
- added REF**: TestPoint_THTPad_D1.5mm_Drill0.7mm, TestPoint:TestPoint_THTPad_D1.5mm_Drill0.7mm, F.Cu at (188.0, 53.3)
- added REF**: TestPoint_THTPad_D1.5mm_Drill0.7mm, TestPoint:TestPoint_THTPad_D1.5mm_Drill0.7mm, F.Cu at (210.8, 106.7)
- added REF**: TestPoint_THTPad_D1.5mm_Drill0.7mm, TestPoint:TestPoint_THTPad_D1.5mm_Drill0.7mm, F.Cu at (208.3, 106.7)
- added REF**: TestPoint_THTPad_D1.5mm_Drill0.7mm, TestPoint:TestPoint_THTPad_D1.5mm_Drill0.7mm, F.Cu at (195.6, 50.8)
- added REF**: TestPoint_THTPad_D1.5mm_Drill0.7mm, TestPoint:TestPoint_THTPad_D1.5mm_Drill0.7mm, F.Cu at (210.8, 104.1)
- added REF**: TestPoint_THTPad_D1.5mm_Drill0.7mm, TestPoint:TestPoint_THTPad_D1.5mm_Drill0.7mm, F.Cu at (167.6, 50.8)
- added REF**: TestPoint_THTPad_D1.5mm_Drill0.7mm, TestPoint:TestPoint_THTPad_D1.5mm_Drill0.7mm, F.Cu at (198.1, 50.8)
- added REF**: TestPoint_THTPad_D1.5mm_Drill0.7mm, TestPoint:TestPoint_THTPad_D1.5mm_Drill0.7mm, F.Cu at (193.0, 96.5)
- added REF**: TestPoint_THTPad_D1.5mm_Drill0.7mm, TestPoint:TestPoint_THTPad_D1.5mm_Drill0.7mm, F.Cu at (185.4, 50.8)
- added REF**: TestPoint_THTPad_D1.5mm_Drill0.7mm, TestPoint:TestPoint_THTPad_D1.5mm_Drill0.7mm, F.Cu at (162.6, 53.3)
- added REF**: TestPoint_THTPad_D1.5mm_Drill0.7mm, TestPoint:TestPoint_THTPad_D1.5mm_Drill0.7mm, F.Cu at (170.2, 50.8)
- added REF**: TestPoint_THTPad_D1.5mm_Drill0.7mm, TestPoint:TestPoint_THTPad_D1.5mm_Drill0.7mm, F.Cu at (208.3, 109.2)
- added REF**: TestPoint_THTPad_D1.5mm_Drill0.7mm, TestPoint:TestPoint_THTPad_D1.5mm_Drill0.7mm, F.Cu at (175.3, 50.8)
- added REF**: TestPoint_THTPad_D1.5mm_Drill0.7mm, TestPoint:TestPoint_THTPad_D1.5mm_Drill0.7mm, F.Cu at (200.7, 106.7)
- added REF**: TestPoint_THTPad_D1.5mm_Drill0.7mm, TestPoint:TestPoint_THTPad_D1.5mm_Drill0.7mm, F.Cu at (190.5, 53.3)
- added REF**: TestPoint_THTPad_D1.5mm_Drill0.7mm, TestPoint:TestPoint_THTPad_D1.5mm_Drill0.7mm, F.Cu at (177.8, 50.8)
- added REF**: TestPoint_THTPad_D1.5mm_Drill0.7mm, TestPoint:TestPoint_THTPad_D1.5mm_Drill0.7mm, F.Cu at (165.1, 50.8)
- added REF**: TestPoint_THTPad_D1.5mm_Drill0.7mm, TestPoint:TestPoint_THTPad_D1.5mm_Drill0.7mm, F.Cu at (162.6, 50.8)
- added REF**: TestPoint_THTPad_D1.5mm_Drill0.7mm, TestPoint:TestPoint_THTPad_D1.5mm_Drill0.7mm, F.Cu at (195.6, 106.7)
- added REF**: TestPoint_THTPad_D1.5mm_Drill0.7mm, TestPoint:TestPoint_THTPad_D1.5mm_Drill0.7mm, F.Cu at (200.7, 104.1)
- added REF**: TestPoint_THTPad_D1.5mm_Drill0.7mm, TestPoint:TestPoint_THTPad_D1.5mm_Drill0.7mm, F.Cu at (147.3, 50.8)
- added REF**: TestPoint_THTPad_D1.5mm_Drill0.7mm, TestPoint:TestPoint_THTPad_D1.5mm_Drill0.7mm, F.Cu at (195.6, 96.5)
- added REF**: TestPoint_THTPad_D1.5mm_Drill0.7mm, TestPoint:TestPoint_THTPad_D1.5mm_Drill0.7mm, F.Cu at (137.2, 50.8)
- added REF**: TestPoint_THTPad_D1.5mm_Drill0.7mm, TestPoint:TestPoint_THTPad_D1.5mm_Drill0.7mm, F.Cu at (190.5, 50.8)
- added REF**: TestPoint_THTPad_D1.5mm_Drill0.7mm, TestPoint:TestPoint_THTPad_D1.5mm_Drill0.7mm, F.Cu at (193.0, 53.3)
- added REF**: TestPoint_THTPad_D1.5mm_Drill0.7mm, TestPoint:TestPoint_THTPad_D1.5mm_Drill0.7mm, F.Cu at (149.9, 53.3)
- added REF**: TestPoint_THTPad_D1.5mm_Drill0.7mm, TestPoint:TestPoint_THTPad_D1.5mm_Drill0.7mm, F.Cu at (198.1, 53.3)
- added REF**: TestPoint_THTPad_D1.5mm_Drill0.7mm, TestPoint:TestPoint_THTPad_D1.5mm_Drill0.7mm, F.Cu at (193.0, 104.1)
- added REF**: TestPoint_THTPad_D1.5mm_Drill0.7mm, TestPoint:TestPoint_THTPad_D1.5mm_Drill0.7mm, F.Cu at (172.7, 53.3)
- added REF**: TestPoint_THTPad_D1.5mm_Drill0.7mm, TestPoint:TestPoint_THTPad_D1.5mm_Drill0.7mm, F.Cu at (160.0, 50.8)
- added REF**: TestPoint_THTPad_D1.5mm_Drill0.7mm, TestPoint:TestPoint_THTPad_D1.5mm_Drill0.7mm, F.Cu at (205.7, 104.1)
- added REF**: TestPoint_THTPad_D1.5mm_Drill0.7mm, TestPoint:TestPoint_THTPad_D1.5mm_Drill0.7mm, F.Cu at (205.7, 111.8)
- added REF**: TestPoint_THTPad_D1.5mm_Drill0.7mm, TestPoint:TestPoint_THTPad_D1.5mm_Drill0.7mm, F.Cu at (157.5, 50.8)
- added REF**: TestPoint_THTPad_D1.5mm_Drill0.7mm, TestPoint:TestPoint_THTPad_D1.5mm_Drill0.7mm, F.Cu at (198.1, 101.6)
- added REF**: TestPoint_THTPad_D1.5mm_Drill0.7mm, TestPoint:TestPoint_THTPad_D1.5mm_Drill0.7mm, F.Cu at (132.1, 50.8)
- added REF**: TestPoint_THTPad_D1.5mm_Drill0.7mm, TestPoint:TestPoint_THTPad_D1.5mm_Drill0.7mm, F.Cu at (190.5, 99.1)
- added REF**: TestPoint_THTPad_D1.5mm_Drill0.7mm, TestPoint:TestPoint_THTPad_D1.5mm_Drill0.7mm, F.Cu at (134.6, 50.8)
- added REF**: TestPoint_THTPad_D1.5mm_Drill0.7mm, TestPoint:TestPoint_THTPad_D1.5mm_Drill0.7mm, F.Cu at (210.8, 109.2)
- added REF**: TestPoint_THTPad_D1.5mm_Drill0.7mm, TestPoint:TestPoint_THTPad_D1.5mm_Drill0.7mm, F.Cu at (195.6, 99.1)
- added REF**: TestPoint_THTPad_D1.5mm_Drill0.7mm, TestPoint:TestPoint_THTPad_D1.5mm_Drill0.7mm, F.Cu at (195.6, 109.2)
- added REF**: TestPoint_THTPad_D1.5mm_Drill0.7mm, TestPoint:TestPoint_THTPad_D1.5mm_Drill0.7mm, F.Cu at (188.0, 50.8)
- added REF**: TestPoint_THTPad_D1.5mm_Drill0.7mm, TestPoint:TestPoint_THTPad_D1.5mm_Drill0.7mm, F.Cu at (147.3, 53.3)
- added REF**: TestPoint_THTPad_D1.5mm_Drill0.7mm, TestPoint:TestPoint_THTPad_D1.5mm_Drill0.7mm, F.Cu at (193.0, 50.8)
- added REF**: TestPoint_THTPad_D1.5mm_Drill0.7mm, TestPoint:TestPoint_THTPad_D1.5mm_Drill0.7mm, F.Cu at (213.4, 109.2)
- added REF**: TestPoint_THTPad_D1.5mm_Drill0.7mm, TestPoint:TestPoint_THTPad_D1.5mm_Drill0.7mm, F.Cu at (193.0, 101.6)
- added REF**: TestPoint_THTPad_D1.5mm_Drill0.7mm, TestPoint:TestPoint_THTPad_D1.5mm_Drill0.7mm, F.Cu at (213.4, 106.7)
- added REF**: TestPoint_THTPad_D1.5mm_Drill0.7mm, TestPoint:TestPoint_THTPad_D1.5mm_Drill0.7mm, F.Cu at (190.5, 109.2)
- added REF**: TestPoint_THTPad_D1.5mm_Drill0.7mm, TestPoint:TestPoint_THTPad_D1.5mm_Drill0.7mm, F.Cu at (142.2, 50.8)
- added REF**: TestPoint_THTPad_D1.5mm_Drill0.7mm, TestPoint:TestPoint_THTPad_D1.5mm_Drill0.7mm, F.Cu at (149.9, 50.8)
- added REF**: TestPoint_THTPad_D1.5mm_Drill0.7mm, TestPoint:TestPoint_THTPad_D1.5mm_Drill0.7mm, F.Cu at (208.3, 104.1)
- added REF**: TestPoint_THTPad_D1.5mm_Drill0.7mm, TestPoint:TestPoint_THTPad_D1.5mm_Drill0.7mm, F.Cu at (180.3, 53.3)
- added REF**: TestPoint_THTPad_D1.5mm_Drill0.7mm, TestPoint:TestPoint_THTPad_D1.5mm_Drill0.7mm, F.Cu at (190.5, 106.7)
- added REF**: TestPoint_THTPad_D1.5mm_Drill0.7mm, TestPoint:TestPoint_THTPad_D1.5mm_Drill0.7mm, F.Cu at (134.6, 53.3)
- added REF**: TestPoint_THTPad_D1.5mm_Drill0.7mm, TestPoint:TestPoint_THTPad_D1.5mm_Drill0.7mm, F.Cu at (198.1, 104.1)
- added REF**: TestPoint_THTPad_D1.5mm_Drill0.7mm, TestPoint:TestPoint_THTPad_D1.5mm_Drill0.7mm, F.Cu at (193.0, 109.2)
- added REF**: TestPoint_THTPad_D1.5mm_Drill0.7mm, TestPoint:TestPoint_THTPad_D1.5mm_Drill0.7mm, F.Cu at (203.2, 53.3)
- added REF**: TestPoint_THTPad_D1.5mm_Drill0.7mm, TestPoint:TestPoint_THTPad_D1.5mm_Drill0.7mm, F.Cu at (200.7, 114.3)
- added REF**: TestPoint_THTPad_D1.5mm_Drill0.7mm, TestPoint:TestPoint_THTPad_D1.5mm_Drill0.7mm, F.Cu at (195.6, 114.3)
- added REF**: TestPoint_THTPad_D1.5mm_Drill0.7mm, TestPoint:TestPoint_THTPad_D1.5mm_Drill0.7mm, F.Cu at (139.7, 50.8)
- added REF**: TestPoint_THTPad_D1.5mm_Drill0.7mm, TestPoint:TestPoint_THTPad_D1.5mm_Drill0.7mm, F.Cu at (190.5, 101.6)
- added REF**: TestPoint_THTPad_D1.5mm_Drill0.7mm, TestPoint:TestPoint_THTPad_D1.5mm_Drill0.7mm, F.Cu at (193.0, 99.1)
- added REF**: TestPoint_THTPad_D1.5mm_Drill0.7mm, TestPoint:TestPoint_THTPad_D1.5mm_Drill0.7mm, F.Cu at (203.2, 109.2)
- added REF**: TestPoint_THTPad_D1.5mm_Drill0.7mm, TestPoint:TestPoint_THTPad_D1.5mm_Drill0.7mm, F.Cu at (144.8, 50.8)
- added REF**: TestPoint_THTPad_D1.5mm_Drill0.7mm, TestPoint:TestPoint_THTPad_D1.5mm_Drill0.7mm, F.Cu at (154.9, 50.8)
- added REF**: TestPoint_THTPad_D1.5mm_Drill0.7mm, TestPoint:TestPoint_THTPad_D1.5mm_Drill0.7mm, F.Cu at (203.2, 50.8)
- added REF**: TestPoint_THTPad_D1.5mm_Drill0.7mm, TestPoint:TestPoint_THTPad_D1.5mm_Drill0.7mm, F.Cu at (152.4, 53.3)
- added REF**: TestPoint_THTPad_D1.5mm_Drill0.7mm, TestPoint:TestPoint_THTPad_D1.5mm_Drill0.7mm, F.Cu at (203.2, 106.7)
- added REF**: TestPoint_THTPad_D1.5mm_Drill0.7mm, TestPoint:TestPoint_THTPad_D1.5mm_Drill0.7mm, F.Cu at (175.3, 53.3)
- added REF**: TestPoint_THTPad_D1.5mm_Drill0.7mm, TestPoint:TestPoint_THTPad_D1.5mm_Drill0.7mm, F.Cu at (193.0, 111.8)
- added REF**: TestPoint_THTPad_D1.5mm_Drill0.7mm, TestPoint:TestPoint_THTPad_D1.5mm_Drill0.7mm, F.Cu at (205.7, 114.3)
- added REF**: TestPoint_THTPad_D1.5mm_Drill0.7mm, TestPoint:TestPoint_THTPad_D1.5mm_Drill0.7mm, F.Cu at (205.7, 50.8)
- added REF**: TestPoint_THTPad_D1.5mm_Drill0.7mm, TestPoint:TestPoint_THTPad_D1.5mm_Drill0.7mm, F.Cu at (177.8, 53.3)
- added REF**: TestPoint_THTPad_D1.5mm_Drill0.7mm, TestPoint:TestPoint_THTPad_D1.5mm_Drill0.7mm, F.Cu at (142.2, 53.3)
- added REF**: TestPoint_THTPad_D1.5mm_Drill0.7mm, TestPoint:TestPoint_THTPad_D1.5mm_Drill0.7mm, F.Cu at (198.1, 114.3)
- added REF**: TestPoint_THTPad_D1.5mm_Drill0.7mm, TestPoint:TestPoint_THTPad_D1.5mm_Drill0.7mm, F.Cu at (195.6, 104.1)
- added REF**: TestPoint_THTPad_D1.5mm_Drill0.7mm, TestPoint:TestPoint_THTPad_D1.5mm_Drill0.7mm, F.Cu at (190.5, 96.5)
- added REF**: TestPoint_THTPad_D1.5mm_Drill0.7mm, TestPoint:TestPoint_THTPad_D1.5mm_Drill0.7mm, F.Cu at (203.2, 111.8)
- added REF**: TestPoint_THTPad_D1.5mm_Drill0.7mm, TestPoint:TestPoint_THTPad_D1.5mm_Drill0.7mm, F.Cu at (205.7, 53.3)
- added REF**: TestPoint_THTPad_D1.5mm_Drill0.7mm, TestPoint:TestPoint_THTPad_D1.5mm_Drill0.7mm, F.Cu at (132.1, 53.3)
- added REF**: TestPoint_THTPad_D1.5mm_Drill0.7mm, TestPoint:TestPoint_THTPad_D1.5mm_Drill0.7mm, F.Cu at (200.7, 50.8)
- added REF**: TestPoint_THTPad_D1.5mm_Drill0.7mm, TestPoint:TestPoint_THTPad_D1.5mm_Drill0.7mm, F.Cu at (190.5, 111.8)
- added REF**: TestPoint_THTPad_D1.5mm_Drill0.7mm, TestPoint:TestPoint_THTPad_D1.5mm_Drill0.7mm, F.Cu at (195.6, 111.8)
- added REF**: TestPoint_THTPad_D1.5mm_Drill0.7mm, TestPoint:TestPoint_THTPad_D1.5mm_Drill0.7mm, F.Cu at (193.0, 106.7)
- added REF**: TestPoint_THTPad_D1.5mm_Drill0.7mm, TestPoint:TestPoint_THTPad_D1.5mm_Drill0.7mm, F.Cu at (144.8, 53.3)
- added REF**: TestPoint_THTPad_D1.5mm_Drill0.7mm, TestPoint:TestPoint_THTPad_D1.5mm_Drill0.7mm, F.Cu at (190.5, 104.1)
- added REF**: TestPoint_THTPad_D1.5mm_Drill0.7mm, TestPoint:TestPoint_THTPad_D1.5mm_Drill0.7mm, F.Cu at (190.5, 114.3)
- added REF**: TestPoint_THTPad_D1.5mm_Drill0.7mm, TestPoint:TestPoint_THTPad_D1.5mm_Drill0.7mm, F.Cu at (167.6, 53.3)
- added REF**: TestPoint_THTPad_D1.5mm_Drill0.7mm, TestPoint:TestPoint_THTPad_D1.5mm_Drill0.7mm, F.Cu at (160.0, 53.3)
- added REF**: TestPoint_THTPad_D1.5mm_Drill0.7mm, TestPoint:TestPoint_THTPad_D1.5mm_Drill0.7mm, F.Cu at (185.4, 53.3)
- added REF**: TestPoint_THTPad_D1.5mm_Drill0.7mm, TestPoint:TestPoint_THTPad_D1.5mm_Drill0.7mm, F.Cu at (172.7, 50.8)
- added REF**: TestPoint_THTPad_D1.5mm_Drill0.7mm, TestPoint:TestPoint_THTPad_D1.5mm_Drill0.7mm, F.Cu at (195.6, 53.3)
- added REF**: TestPoint_THTPad_D1.5mm_Drill0.7mm, TestPoint:TestPoint_THTPad_D1.5mm_Drill0.7mm, F.Cu at (152.4, 50.8)
- added REF**: TestPoint_THTPad_D1.5mm_Drill0.7mm, TestPoint:TestPoint_THTPad_D1.5mm_Drill0.7mm, F.Cu at (198.1, 109.2)
- added REF**: TestPoint_THTPad_D1.5mm_Drill0.7mm, TestPoint:TestPoint_THTPad_D1.5mm_Drill0.7mm, F.Cu at (165.1, 53.3)
- added REF**: TestPoint_THTPad_D1.5mm_Drill0.7mm, TestPoint:TestPoint_THTPad_D1.5mm_Drill0.7mm, F.Cu at (139.7, 53.3)
- moved SW1 5.03 mm to (214.6, 98.0)
- moved J1 4.66 mm to (213.9, 88.0)
- moved PiOLED 0.54 mm to (129.0, 86.0)
- moved J7 0.07 mm to (129.0, 60.6)
- renumbered J8 to PiOLED
Routing:
- net +5V: track 41.7 -> 145.6 mm
- net GND: track 226.3 -> 293.3 mm, vias 0 -> 4
- net +3.3V: track 70.3 -> 131.8 mm, vias 1 -> 0
- net +9V: track 0.00 -> 44.1 mm
- net I2C_2_SDA: track 41.8 -> 79.2 mm, vias 1 -> 2
- net I2C_2_SCL: track 44.1 -> 80.2 mm, vias 1 -> 2
- net Net-(SW1-Pad1): track 0.00 -> 10.6 mm
- added copper zone on F.Cu, net +5V
- added copper zone on B.Cu, net GND
